Commit message: Release_2.3: Add support for 2.3 sensor firmware (IMU / CMV4000 support), add 'MultiSenseUpdater' firmware upgrade tool, add smart dynamic_reconfigure presentation, remove multisense_diagnostics/multisense_dashboard, wire protocol to version 3.0 (w/ support for forthcoming SGM core), misc. other bugfixes and feature enhancements.

File: multisense_description/urdf/multisense.urdf (robot description, URDF)
Before this commit: robot multisense, 25 links, 24 joints
Links:
- added link accel
- added link gyro
- added link mag
Joints:
- added joint accel_joint: type fixed, parent head_root, child accel, origin xyz=-.0475 .0302 -.00275 rpy=0 1.5707 0
- added joint gyro_joint: type fixed, parent head_root, child gyro, origin xyz=-.0476 .0388 -.00075 rpy=1.5707 3.14159 1.5707 
- added joint mag_joint: type fixed, parent head_root, child mag, origin xyz=-.0475 .0302 -.00275 rpy=0 1.5707 0
