Commit message: Add S27 stl model

File: multisense_description/urdf/multisenseS27/multisenseS27.urdf.xacro (robot description, xacro)
@@ -6,5 +6,5 @@
                 <origin xyz="0 0 0" rpy="1.57079632679 0 1.57079632679" />
                 <geometry>
-                    <mesh filename="package://multisense_description/meshes/multisense_s21.STL"/>
+                    <mesh filename="package://multisense_description/meshes/multisense_s27.STL" scale="0.001 0.001 0.001"/>
                 </geometry>
                 <material name="">
@@ -14,5 +14,5 @@
         </link>
         <joint name="${name}/left_camera_joint" type="fixed">
-            <origin xyz="0.0052046 0.105 0" rpy="-1.57079632679 0.0 -1.57079632679"/>
+            <origin xyz="0.08 0.312 0.037" rpy="-1.989 0.0 -1.57079632679"/>
             <parent link="${name}/head"/>
             <child link="${name}/left_camera_frame"/>
