Commit message: Apply TF change to all urdf models

File: multisense_description/urdf/multisenseBCAM/multisenseBCAM.urdf.xacro (robot description, xacro)
@@ -20,8 +20,9 @@
         </joint>
         <link name="${name}/left_camera_frame"/>
-        <joint name="${name}/left_camera_optical_joint" type="fixed">
-            <origin xyz="0 0 0" rpy="-1.57079632679 0.0 -1.57079632679"/>
-            <parent link="${name}/left_camera_frame"/>
-            <child link="${name}/left_camera_optical_frame"/>
+        <!-- Left camera optical frame is treated as the camera origin -->
+        <joint name="${name}/head_optical_joint" type="fixed">
+            <origin xyz="0 0 -0.03" rpy="0.0 -1.57079632679 1.57079632679"/>
+            <parent link="${name}/left_camera_optical_frame"/>
+            <child link="${name}/head"/>
         </joint>
         <link name="${name}/left_camera_optical_frame"/>

File: multisense_description/urdf/multisenseS21/multisenseS21.urdf.xacro (robot description, xacro)
@@ -2,12 +2,4 @@
 <robot xmlns:xacro="http://ros.org/wiki/xacro">
     <xacro:macro name="multisenseS21" params="name">
-        <link name="${name}/left_camera_optical_frame"/>
-        <!-- Note the origin of model is 37.3854mm from the rear mounting plane
-             in the x axis -->
-        <joint name="${name}/head_joint" type="fixed">
-            <origin xyz="0.105 0 -0.0052046" rpy="0.0 -1.57079632679 1.57079632679"/>
-            <parent link="${name}/left_camera_optical_frame"/>
-            <child link="${name}/head"/>
-        </joint>
         <link name="${name}/head">
             <visual>
@@ -21,4 +13,13 @@
             </visual>
         </link>
+        <!-- Note the origin of model is 37.3854mm from the rear mounting plane
+             in the x axis -->
+        <!-- Left camera optical frame is treated as the camera origin -->
+        <joint name="${name}/head_joint" type="fixed">
+            <origin xyz="0.105 0 -0.0052046" rpy="0.0 -1.57079632679 1.57079632679"/>
+            <parent link="${name}/left_camera_optical_frame"/>
+            <child link="${name}/head"/>
+        </joint>
+        <link name="${name}/left_camera_optical_frame"/>
         <joint name="${name}/top_left_rear_mount_joint" type="fixed">
             <origin xyz="-0.0373854 0.1 0.014" rpy="0 0 3.14159"/>

File: multisense_description/urdf/multisenseS27/multisenseS27.urdf.xacro (robot description, xacro)
@@ -13,8 +13,9 @@
             </visual>
         </link>
-        <joint name="${name}/left_camera_joint" type="fixed">
-            <origin xyz="0.08 0.312 0.037" rpy="-1.989 0.0 -1.57079632679"/>
-            <parent link="${name}/head"/>
-            <child link="${name}/left_camera_optical_frame"/>
+        <!-- Left camera optical frame is treated as the camera origin -->
+        <joint name="${name}/head_joint" type="fixed">
+            <origin xyz="0.312 0.06630059527 -0.05807952365" rpy="0.0 -1.989 1.57079632679"/>
+            <parent link="${name}/left_camera_optical_frame"/>
+            <child link="${name}/head"/>
         </joint>
         <link name="${name}/left_camera_optical_frame"/>

File: multisense_description/urdf/multisenseS7/multisenseS7.urdf.xacro (robot description, xacro)
@@ -13,10 +13,11 @@
             </visual>
         </link>
-        <joint name="${name}/left_camera_joint" type="fixed">
-            <origin xyz="0.052 0.035 0.0" rpy="-1.57079632679 0.0 -1.57079632679"/>
-            <parent link="${name}/head"/>
-            <child link="${name}/left_camera_opticial_frame"/>
+        <!-- Left camera optical frame is treated as the camera origin -->
+        <joint name="${name}/head_joint" type="fixed">
+            <origin xyz="0.035 0.0 -0.052" rpy="0.0 -1.57079632679 1.57079632679"/>
+            <parent link="${name}/left_camera_optical_frame"/>
+            <child link="${name}/head"/>
         </joint>
-        <link name="${name}/left_camera_opticial_frame"/>
+        <link name="${name}/left_camera_optical_frame"/>
         <joint name="${name}/accel_joint" type="fixed">
             <origin xyz="0.047 0.0302 -0.00075" rpy="0.0 1.57079632679 0.0"/>

File: multisense_description/urdf/multisenseS7S/multisenseS7S.urdf.xacro (robot description, xacro)
@@ -13,8 +13,9 @@
             </visual>
         </link>
-        <joint name="${name}/left_camera_joint" type="fixed">
-            <origin xyz="0.03 0.035 0.0" rpy="-1.57079632679 0.0 -1.57079632679"/>
-            <parent link="${name}/head"/>
-            <child link="${name}/left_camera_optical_frame"/>
+        <!-- Left camera optical frame is treated as the camera origin -->
+        <joint name="${name}/head_joint" type="fixed">
+            <origin xyz="0.035 0.0 -0.03" rpy="0.0 -1.57079632679 1.57079632679"/>
+            <parent link="${name}/left_camera_optical_frame"/>
+            <child link="${name}/head"/>
         </joint>
         <link name="${name}/left_camera_optical_frame"/>

File: multisense_description/urdf/multisenseSL/multisenseSL.urdf.xacro (robot description, xacro)
@@ -69,10 +69,13 @@
       <child link="${name}/head_hokuyo_frame"/>
     </joint>
-    <!-- Stereo Camera -->
-    <joint name="${name}/left_camera_frame_joint" type="fixed">
+    <!--
+      Stereo Camera
+      Note that the left camera optical frame is treated as the camera origin
+      -->
+    <joint name="${name}/head_joint" type="fixed">
       <!-- optical frame collocated with tilting DOF -->
-      <origin xyz="0.0 0.035 -0.002" rpy="-1.57079632679 0.0 -1.57079632679" />
-      <parent link="${name}/head"/>
-      <child link="${name}/left_camera_optical_frame"/>
+      <origin xyz="0.035 -0.002 0.0" rpy="0.0 -1.57079632679 1.57079632679" />
+      <parent link="${name}/left_camera_optical_frame"/>
+      <child link="${name}/head"/>
     </joint>
     <link name="${name}/left_camera_optical_frame" />
