Commit message: Importable xacro fixes to remove duplicate root frames and fix typos

File: multisense_description/urdf/multisenseBCAM/importable.urdf.xacro (robot description, xacro)
@@ -2,12 +2,6 @@
 <robot xmlns:xacro="http://ros.org/wiki/xacro">
   <xacro:include filename="$(find multisense_description)/urdf/multisenseBCAM/multisenseBCAM.urdf.xacro"/>
-  <xacro:macro name="importable_multisenseBCAM" params="parent name *origin">
-    <!-- Joint for connection to parent -->
-    <joint name="${name}_head_root_joint" type="fixed">
-      <insert_block name="origin"/>
-      <parent link="${parent}"/>
-      <child link="${name}/head"/>
-    </joint>
-    <xacro:multisenseBCAM name="${name}" />
+  <xacro:macro name="importable_multisenseBCAM">
+      <xacro:multisenseBCAM name="${name}" />
   </xacro:macro>
 </robot>

File: multisense_description/urdf/multisenseKS21/importable.urdf.xacro (robot description, xacro)
@@ -2,12 +2,6 @@
 <robot xmlns:xacro="http://ros.org/wiki/xacro">
   <xacro:include filename="$(find multisense_description)/urdf/multisenseKS21/multisenseKS21.urdf.xacro"/>
-  <xacro:macro name="importable_multisenseKS21" params="parent name *origin">
-    <!-- Joint for connection to parent -->
-    <joint name="${name}_head_root_joint" type="fixed">
-      <insert_block name="origin"/>
-      <parent link="${parent}"/>
-      <child link="${name}/head"/>
-    </joint>
-    <xacro:multisenseS27 name="${name}" />
+  <xacro:macro name="importable_multisenseS7">
+      <xacro:multisenseKS21 name="${name}" />
   </xacro:macro>
 </robot>

File: multisense_description/urdf/multisenseS21/importable.urdf.xacro (robot description, xacro)
@@ -2,12 +2,6 @@
 <robot xmlns:xacro="http://ros.org/wiki/xacro">
   <xacro:include filename="$(find multisense_description)/urdf/multisenseS21/multisenseS21.urdf.xacro"/>
-  <xacro:macro name="importable_multisenseS21" params="parent name *origin">
-    <!-- Joint for connection to parent -->
-    <joint name="${name}_head_root_joint" type="fixed">
-      <insert_block name="origin"/>
-      <parent link="${parent}"/>
-      <child link="${name}/head"/>
-    </joint>
-    <xacro:multisenseS21 name="${name}" />
+  <xacro:macro name="importable_multisenseS21">
+      <xacro:multisenseS21 name="${name}" />
   </xacro:macro>
 </robot>

File: multisense_description/urdf/multisenseS7/importable.urdf.xacro (robot description, xacro)
@@ -2,12 +2,6 @@
 <robot xmlns:xacro="http://ros.org/wiki/xacro">
   <xacro:include filename="$(find multisense_description)/urdf/multisenseS7/multisenseS7.urdf.xacro"/>
-  <xacro:macro name="importable_multisenseS7" params="parent name *origin">
-    <!-- Joint for connection to parent -->
-    <joint name="${name}_head_root_joint" type="fixed">
-      <insert_block name="origin"/>
-      <parent link="${parent}"/>
-      <child link="${name}/head"/>
-    </joint>
-    <xacro:multisenseS7 name="${name}" />
+  <xacro:macro name="importable_multisenseS7">
+      <xacro:multisenseS7 name="${name}" />
   </xacro:macro>
 </robot>

File: multisense_description/urdf/multisenseS7S/importable.urdf.xacro (robot description, xacro)
@@ -2,12 +2,6 @@
 <robot xmlns:xacro="http://ros.org/wiki/xacro">
   <xacro:include filename="$(find multisense_description)/urdf/multisenseS7S/multisenseS7S.urdf.xacro"/>
-  <xacro:macro name="importable_multisenseS7S" params="parent name *origin">
-    <!-- Joint for connection to parent -->
-    <joint name="${name}_head_root_joint" type="fixed">
-      <insert_block name="origin"/>
-      <parent link="${parent}"/>
-      <child link="${name}/head"/>
-    </joint>
-    <xacro:multisenseS7S name="${name}" />
+  <xacro:macro name="importable_multisenseS7S">
+      <xacro:multisenseS7S name="${name}" />
   </xacro:macro>
 </robot>

File: multisense_description/urdf/multisenseSL/importable.urdf.xacro (robot description, xacro)
@@ -2,12 +2,6 @@
 <robot xmlns:xacro="http://ros.org/wiki/xacro">
   <xacro:include filename="$(find multisense_description)/urdf/multisenseSL/multisenseSL.urdf.xacro"/>
-  <xacro:macro name="importable_multisenseSL" params="parent name *origin">
-    <!-- Joint for connection to parent -->
-    <joint name="${name}_head_root_joint" type="fixed">
-      <insert_block name="origin"/>
-      <parent link="${parent}"/>
-      <child link="${name}/head"/>
-    </joint>
-    <xacro:multisenseSL name="${name}" />
+  <xacro:macro name="importable_multisenseSL">
+      <xacro:multisenseSL name="${name}" />
   </xacro:macro>
 </robot>
