Commit message: Publish camera extrinsics via a static transform publisher

File: multisense_description/urdf/multisenseS21/multisenseS21.urdf.xacro (robot description, xacro)
@@ -4,5 +4,5 @@
         <link name="${name}/head">
             <visual>
-                <origin xyz="0 0 0" rpy="1.57079632679 0 1.57079632679" />
+                <origin xyz="0.105 0 0" rpy="0 0 3.1415926" />
                 <geometry>
                     <mesh filename="package://multisense_description/meshes/multisense_s21.STL"/>
@@ -13,32 +13,12 @@
             </visual>
         </link>
-        <!-- Note the origin of model is 37.3854mm from the rear mounting plane
-             in the x axis -->
         <joint name="${name}/left_camera_joint" type="fixed">
-            <origin xyz="0.0 0.105 0.0"/>
+            <origin xyz="0.0 0.0 0.0"/>
             <parent link="${name}/head"/>
             <child link="${name}/left_camera_frame"/>
         </joint>
         <link name="${name}/left_camera_frame"/>
-        <joint name="${name}/right_camera_joint" type="fixed">
-            <origin xyz="0.0 -0.105 0.0"/>
-            <parent link="${name}/head"/>
-            <child link="${name}/right_camera_frame"/>
-        </joint>
-        <link name="${name}/right_camera_frame"/>
-        <joint name="${name}/left_camera_optical_joint" type="fixed">
-            <origin xyz="0.0052046 0 0" rpy="-1.57079632679 0.0 -1.57079632679"/>
-            <parent link="${name}/left_camera_frame"/>
-            <child link="${name}/left_camera_optical_frame"/>
-        </joint>
-        <link name="${name}/left_camera_optical_frame"/>
-        <joint name="${name}/right_camera_optical_joint" type="fixed">
-            <origin xyz="0.0052046 0 0" rpy="-1.57079632679 0.0 -1.57079632679"/>
-            <parent link="${name}/right_camera_frame"/>
-            <child link="${name}/right_camera_optical_frame"/>
-        </joint>
-        <link name="${name}/right_camera_optical_frame"/>
         <joint name="${name}/top_left_rear_mount_joint" type="fixed">
-            <origin xyz="-0.0373854 0.1 0.014" rpy="0 0 3.14159"/>
+            <origin xyz="0.005 -0.014 -0.04089" rpy="1.5707963 -1.5707963 0"/>
             <parent link="${name}/head"/>
             <child link="${name}/top_left_rear_mount"/>
@@ -49,5 +29,5 @@
             match the S7/S7S/SL MultiSense configurations -->
         <joint name="${name}/accel_joint" type="fixed">
-            <origin xyz="0.0045 0.029 -0.0135" rpy="0.0 1.57079632679 0.0"/>
+            <origin xyz="0.076 0.0135 -0.0047" rpy="0.0 0.0 0.0"/>
             <parent link="${name}/head"/>
             <child link="${name}/accel"/>
@@ -55,5 +35,5 @@
         <link name="${name}/accel"/>
         <joint name="${name}/mag_joint" type="fixed">
-            <origin xyz="0.0045 0.029 -0.0135" rpy="0.0 1.57079632679 0.0"/>
+            <origin xyz="0.076 0.0135 -0.0047" rpy="0.0 0.0 0.0"/>
             <parent link="${name}/head"/>
             <child link="${name}/mag"/>
@@ -61,5 +41,5 @@
         <link name="${name}/mag"/>
         <joint name="${name}/gyro_joint" type="fixed">
-            <origin xyz="-0.00219539 0.03758 -0.014" rpy="-1.57079632679 0 -1.57079632679"/>
+            <origin xyz="0.0672 0.014 -0.0074" rpy="0.0 3.14159 0.0"/>
             <parent link="${name}/head"/>
             <child link="${name}/gyro"/>

File: multisense_description/urdf/multisenseS7/multisenseS7.urdf.xacro (robot description, xacro)
@@ -4,5 +4,5 @@
         <link name="${name}/head">
             <visual>
-                <origin xyz="-0.03 -0.0625 -0.032" rpy="1.57079632679 0 1.57079632679" />
+                <origin xyz="0.0975 0.0325 -0.047" rpy="0 0 3.1415926" />
                 <geometry>
                     <mesh filename="package://multisense_description/meshes/multisense_s7.STL" scale="0.001 0.001 0.001"/>
@@ -14,27 +14,9 @@
         </link>
         <joint name="${name}/left_camera_joint" type="fixed">
-            <origin xyz="0.052 0.035 0.0"/>
+            <origin xyz="0.0 0.0 0.0"/>
             <parent link="${name}/head"/>
             <child link="${name}/left_camera_frame"/>
         </joint>
         <link name="${name}/left_camera_frame"/>
-        <joint name="${name}/right_camera_joint" type="fixed">
-            <origin xyz="0.052 -0.035 0.0"/>
-            <parent link="${name}/head"/>
-            <child link="${name}/right_camera_frame"/>w
-        </joint>
-        <link name="${name}/right_camera_frame"/>
-        <joint name="${name}/left_camera_optical_joint" type="fixed">
-            <origin xyz="0 0 0" rpy="-1.57079632679 0.0 -1.57079632679"/>
-            <parent link="${name}/left_camera_frame"/>
-            <child link="${name}/left_camera_optical_frame"/>
-        </joint>
-        <link name="${name}/left_camera_optical_frame"/>
-        <joint name="${name}/right_camera_optical_joint" type="fixed">
-            <origin xyz="0 0 0" rpy="-1.57079632679 0.0 -1.57079632679"/>
-            <parent link="${name}/right_camera_frame"/>
-            <child link="${name}/right_camera_optical_frame"/>
-        </joint>
-        <link name="${name}/right_camera_optical_frame"/>
         <joint name="${name}/accel_joint" type="fixed">
             <origin xyz="0.047 0.0302 -0.00075" rpy="0.0 1.57079632679 0.0"/>

File: multisense_description/urdf/multisenseS7S/multisenseS7S.urdf.xacro (robot description, xacro)
@@ -4,5 +4,5 @@
         <link name="${name}/head">
             <visual>
-                <origin xyz="0 -0.0625 -0.037" rpy="1.57079632679 0 1.57079632679" />
+                <origin xyz="0.0975 0.0325 -0.047" rpy="0 0 3.1415926" />
                 <geometry>
                     <mesh filename="package://multisense_description/meshes/multisense_s7s.STL" scale="0.001 0.001 0.001"/>
@@ -14,27 +14,9 @@
         </link>
         <joint name="${name}/left_camera_joint" type="fixed">
-            <origin xyz="0.03 0.035 0.0"/>
+            <origin xyz="0.0 0.0 0.0"/>
             <parent link="${name}/head"/>
             <child link="${name}/left_camera_frame"/>
         </joint>
         <link name="${name}/left_camera_frame"/>
-        <joint name="${name}/right_camera_joint" type="fixed">
-            <origin xyz="0.03 -0.035 0.0"/>
-            <parent link="${name}/head"/>
-            <child link="${name}/right_camera_frame"/>
-        </joint>
-        <link name="${name}/right_camera_frame"/>
-        <joint name="${name}/left_camera_optical_joint" type="fixed">
-            <origin xyz="0 0 0" rpy="-1.57079632679 0.0 -1.57079632679"/>
-            <parent link="${name}/left_camera_frame"/>
-            <child link="${name}/left_camera_optical_frame"/>
-        </joint>
-        <link name="${name}/left_camera_optical_frame"/>
-        <joint name="${name}/right_camera_optical_joint" type="fixed">
-            <origin xyz="0 0 0" rpy="-1.57079632679 0.0 -1.57079632679"/>
-            <parent link="${name}/right_camera_frame"/>
-            <child link="${name}/right_camera_optical_frame"/>
-        </joint>
-        <link name="${name}/right_camera_optical_frame"/>
         <joint name="${name}/accel_joint" type="fixed">
             <origin xyz="0.047 0.0302 -0.00075" rpy="0.0 1.57079632679 0.0"/>

Commit message: Revert URDF changes

File: multisense_description/urdf/multisenseS21/multisenseS21.urdf.xacro (robot description, xacro)
@@ -4,5 +4,5 @@
         <link name="${name}/head">
             <visual>
-                <origin xyz="0.105 0 0" rpy="0 0 3.1415926" />
+                <origin xyz="0 0 0" rpy="1.57079632679 0 1.57079632679" />
                 <geometry>
                     <mesh filename="package://multisense_description/meshes/multisense_s21.STL"/>
@@ -13,6 +13,8 @@
             </visual>
         </link>
+        <!-- Note the origin of model is 37.3854mm from the rear mounting plane
+             in the x axis -->
         <joint name="${name}/left_camera_joint" type="fixed">
-            <origin xyz="0.0 0.0 0.0"/>
+            <origin xyz="0.0052046 0.105 0" rpy="-1.57079632679 0.0 -1.57079632679"/>
             <parent link="${name}/head"/>
             <child link="${name}/left_camera_frame"/>
@@ -20,5 +22,5 @@
         <link name="${name}/left_camera_frame"/>
         <joint name="${name}/top_left_rear_mount_joint" type="fixed">
-            <origin xyz="0.005 -0.014 -0.04089" rpy="1.5707963 -1.5707963 0"/>
+            <origin xyz="-0.0373854 0.1 0.014" rpy="0 0 3.14159"/>
             <parent link="${name}/head"/>
             <child link="${name}/top_left_rear_mount"/>
@@ -29,5 +31,5 @@
             match the S7/S7S/SL MultiSense configurations -->
         <joint name="${name}/accel_joint" type="fixed">
-            <origin xyz="0.076 0.0135 -0.0047" rpy="0.0 0.0 0.0"/>
+            <origin xyz="0.0045 0.029 -0.0135" rpy="0.0 1.57079632679 0.0"/>
             <parent link="${name}/head"/>
             <child link="${name}/accel"/>
@@ -35,5 +37,5 @@
         <link name="${name}/accel"/>
         <joint name="${name}/mag_joint" type="fixed">
-            <origin xyz="0.076 0.0135 -0.0047" rpy="0.0 0.0 0.0"/>
+            <origin xyz="0.0045 0.029 -0.0135" rpy="0.0 1.57079632679 0.0"/>
             <parent link="${name}/head"/>
             <child link="${name}/mag"/>
@@ -41,5 +43,5 @@
         <link name="${name}/mag"/>
         <joint name="${name}/gyro_joint" type="fixed">
-            <origin xyz="0.0672 0.014 -0.0074" rpy="0.0 3.14159 0.0"/>
+            <origin xyz="-0.00219539 0.03758 -0.014" rpy="-1.57079632679 0 -1.57079632679"/>
             <parent link="${name}/head"/>
             <child link="${name}/gyro"/>

File: multisense_description/urdf/multisenseS27/multisenseS27.urdf.xacro (robot description, xacro)
@@ -4,5 +4,5 @@
         <link name="${name}/head">
             <visual>
-                <origin xyz="0 0 0" rpy="0 0 0" />
+                <origin xyz="0 0 0" rpy="1.57079632679 0 1.57079632679" />
                 <geometry>
                     <mesh filename="package://multisense_description/meshes/multisense_s21.STL"/>
@@ -14,5 +14,5 @@
         </link>
         <joint name="${name}/left_camera_joint" type="fixed">
-            <origin xyz="0.0 0.105 0.0"/>
+            <origin xyz="0.0052046 0.105 0" rpy="-1.57079632679 0.0 -1.57079632679"/>
             <parent link="${name}/head"/>
             <child link="${name}/left_camera_frame"/>

File: multisense_description/urdf/multisenseS7/multisenseS7.urdf.xacro (robot description, xacro)
@@ -4,5 +4,5 @@
         <link name="${name}/head">
             <visual>
-                <origin xyz="0.0975 0.0325 -0.047" rpy="0 0 3.1415926" />
+                <origin xyz="-0.03 -0.0625 -0.032" rpy="1.57079632679 0 1.57079632679" />
                 <geometry>
                     <mesh filename="package://multisense_description/meshes/multisense_s7.STL" scale="0.001 0.001 0.001"/>
@@ -14,5 +14,5 @@
         </link>
         <joint name="${name}/left_camera_joint" type="fixed">
-            <origin xyz="0.0 0.0 0.0"/>
+            <origin xyz="0.052 0.035 0.0" rpy="-1.57079632679 0.0 -1.57079632679"/>
             <parent link="${name}/head"/>
             <child link="${name}/left_camera_frame"/>

File: multisense_description/urdf/multisenseS7S/multisenseS7S.urdf.xacro (robot description, xacro)
@@ -4,5 +4,5 @@
         <link name="${name}/head">
             <visual>
-                <origin xyz="0.0975 0.0325 -0.047" rpy="0 0 3.1415926" />
+                <origin xyz="0 -0.0625 -0.037" rpy="1.57079632679 0 1.57079632679" />
                 <geometry>
                     <mesh filename="package://multisense_description/meshes/multisense_s7s.STL" scale="0.001 0.001 0.001"/>
@@ -14,5 +14,5 @@
         </link>
         <joint name="${name}/left_camera_joint" type="fixed">
-            <origin xyz="0.0 0.0 0.0"/>
+            <origin xyz="0.03 0.035 0.0" rpy="-1.57079632679 0.0 -1.57079632679"/>
             <parent link="${name}/head"/>
             <child link="${name}/left_camera_frame"/>

Commit message: Make the left_camera_optical_frame the root of the local sensor tf tree

File: multisense_description/urdf/multisenseS21/multisenseS21.urdf.xacro (robot description, xacro)
@@ -18,7 +18,7 @@
             <origin xyz="0.0052046 0.105 0" rpy="-1.57079632679 0.0 -1.57079632679"/>
             <parent link="${name}/head"/>
-            <child link="${name}/left_camera_frame"/>
+            <child link="${name}/left_camera_optical_frame"/>
         </joint>
-        <link name="${name}/left_camera_frame"/>
+        <link name="${name}/left_camera_optical_frame"/>
         <joint name="${name}/top_left_rear_mount_joint" type="fixed">
             <origin xyz="-0.0373854 0.1 0.014" rpy="0 0 3.14159"/>

File: multisense_description/urdf/multisenseS27/multisenseS27.urdf.xacro (robot description, xacro)
@@ -16,7 +16,7 @@
             <origin xyz="0.08 0.312 0.037" rpy="-1.989 0.0 -1.57079632679"/>
             <parent link="${name}/head"/>
-            <child link="${name}/left_camera_frame"/>
+            <child link="${name}/left_camera_optical_frame"/>
         </joint>
-        <link name="${name}/left_camera_frame"/>
+        <link name="${name}/left_camera_optical_frame"/>
     </xacro:macro>
 </robot>

File: multisense_description/urdf/multisenseS7/multisenseS7.urdf.xacro (robot description, xacro)
@@ -16,7 +16,7 @@
             <origin xyz="0.052 0.035 0.0" rpy="-1.57079632679 0.0 -1.57079632679"/>
             <parent link="${name}/head"/>
-            <child link="${name}/left_camera_frame"/>
+            <child link="${name}/left_camera_opticial_frame"/>
         </joint>
-        <link name="${name}/left_camera_frame"/>
+        <link name="${name}/left_camera_opticial_frame"/>
         <joint name="${name}/accel_joint" type="fixed">
             <origin xyz="0.047 0.0302 -0.00075" rpy="0.0 1.57079632679 0.0"/>

File: multisense_description/urdf/multisenseS7S/multisenseS7S.urdf.xacro (robot description, xacro)
@@ -16,7 +16,7 @@
             <origin xyz="0.03 0.035 0.0" rpy="-1.57079632679 0.0 -1.57079632679"/>
             <parent link="${name}/head"/>
-            <child link="${name}/left_camera_frame"/>
+            <child link="${name}/left_camera_optical_frame"/>
         </joint>
-        <link name="${name}/left_camera_frame"/>
+        <link name="${name}/left_camera_optical_frame"/>
         <joint name="${name}/accel_joint" type="fixed">
             <origin xyz="0.047 0.0302 -0.00075" rpy="0.0 1.57079632679 0.0"/>

Commit message: Major ROS driver refactor to support S27 (#7)
* Major ROS driver refactor to support S27

* Fix build warnings. Add in basic AUX camera support

* Merge fixes

* Add support for aux/rectified aux streams

* Remove boost dependency

* Update color pointcloud streams to support Aux cameras

* Up max S27 framerate

* Confirm config is properly set

* Basic cmake cleanup

* Fix build errors under melodic and kinetic

* Handle invalid aux camera calibrations

* Fix scaling issue with aux camera info

* Refactor to reserve buffers independent of color conversion

* Publish camera extrinsics via a static transform publisher

* Revert URDF changes

* Fix SL URDF. Default to S21 for sensor model

* Add aux mono and mono rect topics

* Add S27 stl model

* Make the left_camera_optical_frame the root of the local sensor tf tree

* Fix urdf for MultiSense SL

* Fix melodic build issues

* crop mode calibration scaling fixes

* Remove dead code

Co-authored-by: QuentinTorg <quentin.torgerson@gmail.com>

File: multisense_description/urdf/multisenseS21/multisenseS21.urdf.xacro (robot description, xacro)
@@ -16,27 +16,9 @@
              in the x axis -->
         <joint name="${name}/left_camera_joint" type="fixed">
-            <origin xyz="0.0 0.105 0.0"/>
+            <origin xyz="0.0052046 0.105 0" rpy="-1.57079632679 0.0 -1.57079632679"/>
             <parent link="${name}/head"/>
-            <child link="${name}/left_camera_frame"/>
-        </joint>
-        <link name="${name}/left_camera_frame"/>
-        <joint name="${name}/right_camera_joint" type="fixed">
-            <origin xyz="0.0 -0.105 0.0"/>
-            <parent link="${name}/head"/>
-            <child link="${name}/right_camera_frame"/>
-        </joint>
-        <link name="${name}/right_camera_frame"/>
-        <joint name="${name}/left_camera_optical_joint" type="fixed">
-            <origin xyz="0.0052046 0 0" rpy="-1.57079632679 0.0 -1.57079632679"/>
-            <parent link="${name}/left_camera_frame"/>
             <child link="${name}/left_camera_optical_frame"/>
         </joint>
         <link name="${name}/left_camera_optical_frame"/>
-        <joint name="${name}/right_camera_optical_joint" type="fixed">
-            <origin xyz="0.0052046 0 0" rpy="-1.57079632679 0.0 -1.57079632679"/>
-            <parent link="${name}/right_camera_frame"/>
-            <child link="${name}/right_camera_optical_frame"/>
-        </joint>
-        <link name="${name}/right_camera_optical_frame"/>
         <joint name="${name}/top_left_rear_mount_joint" type="fixed">
             <origin xyz="-0.0373854 0.1 0.014" rpy="0 0 3.14159"/>

File: multisense_description/urdf/multisenseS7/multisenseS7.urdf.xacro (robot description, xacro)
@@ -14,27 +14,9 @@
         </link>
         <joint name="${name}/left_camera_joint" type="fixed">
-            <origin xyz="0.052 0.035 0.0"/>
+            <origin xyz="0.052 0.035 0.0" rpy="-1.57079632679 0.0 -1.57079632679"/>
             <parent link="${name}/head"/>
-            <child link="${name}/left_camera_frame"/>
+            <child link="${name}/left_camera_opticial_frame"/>
         </joint>
-        <link name="${name}/left_camera_frame"/>
-        <joint name="${name}/right_camera_joint" type="fixed">
-            <origin xyz="0.052 -0.035 0.0"/>
-            <parent link="${name}/head"/>
-            <child link="${name}/right_camera_frame"/>w
-        </joint>
-        <link name="${name}/right_camera_frame"/>
-        <joint name="${name}/left_camera_optical_joint" type="fixed">
-            <origin xyz="0 0 0" rpy="-1.57079632679 0.0 -1.57079632679"/>
-            <parent link="${name}/left_camera_frame"/>
-            <child link="${name}/left_camera_optical_frame"/>
-        </joint>
-        <link name="${name}/left_camera_optical_frame"/>
-        <joint name="${name}/right_camera_optical_joint" type="fixed">
-            <origin xyz="0 0 0" rpy="-1.57079632679 0.0 -1.57079632679"/>
-            <parent link="${name}/right_camera_frame"/>
-            <child link="${name}/right_camera_optical_frame"/>
-        </joint>
-        <link name="${name}/right_camera_optical_frame"/>
+        <link name="${name}/left_camera_opticial_frame"/>
         <joint name="${name}/accel_joint" type="fixed">
             <origin xyz="0.047 0.0302 -0.00075" rpy="0.0 1.57079632679 0.0"/>

File: multisense_description/urdf/multisenseS7S/multisenseS7S.urdf.xacro (robot description, xacro)
@@ -14,27 +14,9 @@
         </link>
         <joint name="${name}/left_camera_joint" type="fixed">
-            <origin xyz="0.03 0.035 0.0"/>
+            <origin xyz="0.03 0.035 0.0" rpy="-1.57079632679 0.0 -1.57079632679"/>
             <parent link="${name}/head"/>
-            <child link="${name}/left_camera_frame"/>
-        </joint>
-        <link name="${name}/left_camera_frame"/>
-        <joint name="${name}/right_camera_joint" type="fixed">
-            <origin xyz="0.03 -0.035 0.0"/>
-            <parent link="${name}/head"/>
-            <child link="${name}/right_camera_frame"/>
-        </joint>
-        <link name="${name}/right_camera_frame"/>
-        <joint name="${name}/left_camera_optical_joint" type="fixed">
-            <origin xyz="0 0 0" rpy="-1.57079632679 0.0 -1.57079632679"/>
-            <parent link="${name}/left_camera_frame"/>
             <child link="${name}/left_camera_optical_frame"/>
         </joint>
         <link name="${name}/left_camera_optical_frame"/>
-        <joint name="${name}/right_camera_optical_joint" type="fixed">
-            <origin xyz="0 0 0" rpy="-1.57079632679 0.0 -1.57079632679"/>
-            <parent link="${name}/right_camera_frame"/>
-            <child link="${name}/right_camera_optical_frame"/>
-        </joint>
-        <link name="${name}/right_camera_optical_frame"/>
         <joint name="${name}/accel_joint" type="fixed">
             <origin xyz="0.047 0.0302 -0.00075" rpy="0.0 1.57079632679 0.0"/>

File: multisense_description/urdf/multisenseSL/multisenseSL.urdf.xacro (robot description, xacro)
@@ -4,9 +4,4 @@
     <!-- Head Link Simplified Collision Mesh -->
     <link name="${name}/head">
-      <inertial>
-        <origin xyz="-0.075493 3.3383E-05 0.02774" rpy="0 0 0" />
-        <mass value="1.4199" />
-        <inertia iyy="0.0041178" ixy="-1.5797E-06" iyz="-6.8415E-07" ixx="0.0039688" ixz="-0.00089293" izz="0.0035243" />
-      </inertial>
       <visual>
         <origin xyz="0 0  0" rpy="0 0 0" />
@@ -77,39 +72,9 @@
     <joint name="${name}/left_camera_frame_joint" type="fixed">
       <!-- optical frame collocated with tilting DOF -->
-      <origin xyz="0.0 0.035 -0.002"/>
+      <origin xyz="0.0 0.035 -0.002" rpy="-1.57079632679 0.0 -1.57079632679" />
       <parent link="${name}/head"/>
-      <child link="${name}/left_camera_frame"/>
-    </joint>
-    <link name="${name}/left_camera_frame">
-      <inertial>
-        <mass value="0.1" />
-        <origin xyz="0 0 0" />
-        <inertia ixx="0.001"  ixy="0.0"  ixz="0.0" iyy="0.001"  iyz="0.0" izz="0.001" />
-      </inertial>
-    </link>
-    <joint name="${name}/left_camera_optical_frame_joint" type="fixed">
-      <origin xyz="0 0 0" rpy="-1.57079632679 0.0 -1.57079632679" />
-      <parent link="${name}/left_camera_frame" />
       <child link="${name}/left_camera_optical_frame"/>
     </joint>
-    <link name="${name}/left_camera_optical_frame"/>
-    <joint name="${name}/right_camera_frame_joint" type="fixed">
-      <origin xyz="0.0 -0.035 -0.002"/>
-      <parent link="${name}/head"/>
-      <child link="${name}/right_camera_frame"/>
-    </joint>
-    <link name="${name}/right_camera_frame">
-      <inertial>
-        <mass value="0.1" />
-        <origin xyz="0 0 0" />
-        <inertia ixx="0.001"  ixy="0.0"  ixz="0.0" iyy="0.001"  iyz="0.0" izz="0.001" />
-      </inertial>
-    </link>
-    <joint name="${name}/right_camera_optical_frame_joint" type="fixed">
-      <origin xyz="0 0 0" rpy="-1.5708 0.0 -1.5708" />
-      <parent link="${name}/right_camera_frame" />
-      <child link="${name}/right_camera_optical_frame"/>
-    </joint>
-    <link name="${name}/right_camera_optical_frame"/>
+    <link name="${name}/left_camera_optical_frame" />
     <joint name="${name}/center_top_led_frame_joint" type="fixed">
       <origin xyz="0.01125 0.0 0.0105"/>
