Commit message: Modify TF tree hierarchy

File: multisense_description/urdf/multisenseS21/multisenseS21.urdf.xacro (robot description, xacro)
@@ -2,4 +2,12 @@
 <robot xmlns:xacro="http://ros.org/wiki/xacro">
     <xacro:macro name="multisenseS21" params="name">
+        <link name="${name}/left_camera_optical_frame"/>
+        <!-- Note the origin of model is 37.3854mm from the rear mounting plane
+             in the x axis -->
+        <joint name="${name}/head_joint" type="fixed">
+            <origin xyz="0.105 0 -0.0052046" rpy="0.0 -1.57079632679 1.57079632679"/>
+            <parent link="${name}/left_camera_optical_frame"/>
+            <child link="${name}/head"/>
+        </joint>
         <link name="${name}/head">
             <visual>
@@ -13,12 +21,4 @@
             </visual>
         </link>
-        <!-- Note the origin of model is 37.3854mm from the rear mounting plane
-             in the x axis -->
-        <joint name="${name}/left_camera_joint" type="fixed">
-            <origin xyz="0.0052046 0.105 0" rpy="-1.57079632679 0.0 -1.57079632679"/>
-            <parent link="${name}/head"/>
-            <child link="${name}/left_camera_optical_frame"/>
-        </joint>
-        <link name="${name}/left_camera_optical_frame"/>
         <joint name="${name}/top_left_rear_mount_joint" type="fixed">
             <origin xyz="-0.0373854 0.1 0.014" rpy="0 0 3.14159"/>

Commit message: Support dynamic extrinsics parameter updates (#34)
Add support to ROS driver to modify extrinsics. The reconfigure callback updates the 
extrinsics on-board the multisense — this is important to tools such as ground surface 
modelling which run on the camera and rely on these extrinsics being set correctly. 
The callback also updates a transform member in the camera class, which allows the 
user to dynamically redraw the pointcloud position in the RVIZ window.

File: multisense_description/urdf/multisenseS21/multisenseS21.urdf.xacro (robot description, xacro)
@@ -15,8 +15,9 @@
         <!-- Note the origin of model is 37.3854mm from the rear mounting plane
              in the x axis -->
-        <joint name="${name}/left_camera_joint" type="fixed">
-            <origin xyz="0.0052046 0.105 0" rpy="-1.57079632679 0.0 -1.57079632679"/>
-            <parent link="${name}/head"/>
-            <child link="${name}/left_camera_optical_frame"/>
+        <!-- Left camera optical frame is treated as the camera origin -->
+        <joint name="${name}/head_joint" type="fixed">
+            <origin xyz="0.105 0 -0.0052046" rpy="0.0 -1.57079632679 1.57079632679"/>
+            <parent link="${name}/left_camera_optical_frame"/>
+            <child link="${name}/head"/>
         </joint>
         <link name="${name}/left_camera_optical_frame"/>
