Commit message: fix the urdf issues on launch caused by incorrect file paths and names

File: multisense_description/urdf/multisenseremote_head_monocam/importable.urdf.xacro (robot description, xacro)
@@ -1,6 +1,6 @@
 <?xml version="1.0" ?>
 <robot xmlns:xacro="http://ros.org/wiki/xacro">
-  <xacro:include filename="$(find multisense_description)/urdf/multisensemultisense_remote_head_stereo/multisense_remote_head_stereo.urdf.xacro"/>
-  <xacro:macro name="importable_multisense_remote_head_stereo" params="parent name *origin">
+  <xacro:include filename="$(find multisense_description)/urdf/multisenseremote_head_monocam/multisense_remote_head_monocam.urdf.xacro"/>
+  <xacro:macro name="importable_multisense_remote_head_monocam" params="parent name *origin">
     <!-- Joint for connection to parent -->
     <joint name="${name}_head_root_joint" type="fixed">
@@ -9,5 +9,5 @@
       <child link="${name}/head"/>
     </joint>
-    <xacro:multisense_remote_head_stereo name="${name}" />
+    <xacro:multisense_remote_head_monocam name="${name}" />
   </xacro:macro>
 </robot>

File: multisense_description/urdf/multisenseremote_head_stereo/importable.urdf.xacro (robot description, xacro)
@@ -1,6 +1,6 @@
 <?xml version="1.0" ?>
 <robot xmlns:xacro="http://ros.org/wiki/xacro">
-  <xacro:include filename="$(find multisense_description)/urdf/multisense_remote_head_monocam/multisense_remote_head_monocam.urdf.xacro"/>
-  <xacro:macro name="importable_multisense_remote_head_monocam" params="parent name *origin">
+  <xacro:include filename="$(find multisense_description)/urdf/multisenseremote_head_stereo/multisense_remote_head_stereo.urdf.xacro"/>
+  <xacro:macro name="importable_multisense_remote_head_stereo" params="parent name *origin">
     <!-- Joint for connection to parent -->
     <joint name="${name}_head_root_joint" type="fixed">
@@ -9,5 +9,5 @@
       <child link="${name}/head"/>
     </joint>
-    <xacro:multisense_remote_head_monocam name="${name}" />
+    <xacro:multisense_remote_head_stereo name="${name}" />
   </xacro:macro>
 </robot>

File: multisense_description/urdf/multisenseremote_head_stereo/standalone.urdf.xacro (robot description, xacro)
@@ -1,4 +1,4 @@
 <robot name="multisense" xmlns:xacro="http://ros.org/wiki/xacro">
-    <xacro:include filename="$(find multisense_description)/urdf/multisense_remote_head_stereo/multisense_remote_head_stereo.urdf.xacro"/>
+    <xacro:include filename="$(find multisense_description)/urdf/multisenseremote_head_stereo/multisense_remote_head_stereo.urdf.xacro"/>
     <xacro:multisense_remote_head_stereo name="$(arg name)"/>
 </robot>

File: multisense_description/urdf/multisenseremote_head_vpb/importable.urdf.xacro (robot description, xacro)
@@ -1,5 +1,5 @@
 <?xml version="1.0" ?>
 <robot xmlns:xacro="http://ros.org/wiki/xacro">
-  <xacro:include filename="$(find multisense_description)/urdf/multisense_remote_head_vpb/multisense_remote_head_vpb.urdf.xacro"/>
+  <xacro:include filename="$(find multisense_description)/urdf/multisenseremote_head_vpb/multisense_remote_head_vpb.urdf.xacro"/>
   <xacro:macro name="importable_multisense_remote_head_vpb" params="parent name *origin">
     <!-- Joint for connection to parent -->

File: multisense_description/urdf/multisenseremote_head_vpb/standalone.urdf.xacro (robot description, xacro)
@@ -1,4 +1,4 @@
 <robot name="multisense" xmlns:xacro="http://ros.org/wiki/xacro">
-    <xacro:include filename="$(find multisense_description)/urdf/multisense_remote_head_vpb/multisense_remote_head_vpb.urdf.xacro"/>
+    <xacro:include filename="$(find multisense_description)/urdf/multisenseremote_head_vpb/multisense_remote_head_vpb.urdf.xacro"/>
     <xacro:multisense_remote_head_vpb name="$(arg name)"/>
 </robot>
