Commit message: Update the S30 processor board IMU location

File: multisense_description/urdf/multisenseS30/multisenseS30.urdf.xacro (robot description, xacro)
@@ -21,5 +21,5 @@
         <link name="${name}/imu"/>
         <joint name="${name}/imu_joint" type="fixed">
-            <origin xyz="0.0873 0.0074 -0.0371" rpy="1.57079632679 0.0 0.0"/>
+            <origin xyz="0.494 -0.0063 -0.042" rpy="-1.57079632679 0.0 0.0"/>
             <parent link="${name}/left_camera_optical_frame"/>
             <child link="${name}/imu"/>
