Commit message: update the s21b xacro to match naming from other sensors

File: multisense_description/urdf/multisenseS21B/multisenseS21B.urdf.xacro (robot description, xacro)
@@ -1,5 +1,5 @@
 <?xml version="1.0" ?>
 <robot xmlns:xacro="http://ros.org/wiki/xacro">
-    <xacro:macro name="multisenseS21b" params="name">
+    <xacro:macro name="multisenseS21B" params="name">
         <link name="${name}/head">
             <visual>
@@ -21,5 +21,5 @@
         <link name="${name}/left_camera_optical_frame"/>
         <!--Note the locations of the accel/mag and gyro differ from those shown
-            in CAD. The S21 firmware switches axis on the accel/mag and gyro to
+            in CAD. The S21B firmware switches axis on the accel/mag and gyro to
             match the S7/S7S/SL MultiSense configurations -->
         <joint name="${name}/accel_joint" type="fixed">

File: multisense_description/urdf/multisenseS21B/standalone.urdf.xacro (robot description, xacro)
@@ -1,4 +1,4 @@
 <robot name="multisense" xmlns:xacro="http://ros.org/wiki/xacro">
-    <xacro:include filename="$(find multisense_description)/urdf/multisenseS21B/multisenseS21b.urdf.xacro"/>
-    <xacro:multisenseS21b name="$(arg name)"/>
+    <xacro:include filename="$(find multisense_description)/urdf/multisenseS21B/multisenseS21B.urdf.xacro"/>
+    <xacro:multisenseS21B name="$(arg name)"/>
 </robot>
